File: schematic/plankStrap/plankStrap.kicad_sch (KiCad schematic)
At the start: 3 parts, among them U1 Xplained_328p, U2 Gyro_Absolute_BNO055, U3 LCD_2.4in_ILI9341

Commit message: fixed schematic again
Other:
- note added: "Output in Eueler angles"
- moved on the sheet: U2
Changed lines of the file:
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@@
+		)
+	)
+	(text "Output in Eueler angles"
+		(exclude_from_sim no)
+		(at 216.154 38.608 0)
+		(effects
+			(font
+				(size 3 3)
+			)
 		)
 	)
@@
 	)
 	(no_connect
-		(at 128.27 62.23)
+		(at 125.73 58.42)
 	)
 	(no_connect
-		(at 151.13 52.07)
+		(at 148.59 48.26)
 	)
 	(no_connect
-		(at 137.16 44.45)
+		(at 134.62 40.64)
 	)
 	(no_connect
@@
 	)
 	(no_connect
-		(at 151.13 63.5)
+		(at 148.59 59.69)
 	)
 	(no_connect
-		(at 151.13 55.88)
+		(at 148.59 52.07)
 	)
 	(global_label "DC"
@@
 	(global_label "GND"
 		(shape input)
-		(at 139.7 71.12 270)
-		(fields_autoplaced yes)
-		(effects
-			(font
-				(size 1.27 1.27)
-			)
-			(justify right)
-		)
-		(property "Intersheetrefs" "${INTERSHEET_REFS}"
-			(at 139.7 77.9757 90)
+		(at 137.16 67.31 270)
+		(fields_autoplaced yes)
+		(effects
+			(font
+				(size 1.27 1.27)
+			)
+			(justify right)
+		)
+		(property "Intersheetrefs" "${INTERSHEET_REFS}"
+			(at 137.16 74.1657 90)
 			(effects
 				(font
@@
 	(global_label "SCL"
 		(shape input)
-		(at 128.27 58.42 180)
-		(fields_autoplaced yes)
-		(effects
-			(font
-				(size 1.27 1.27)
-			)
-			(justify right)
-		)
-		(property "Intersheetrefs" "${INTERSHEET_REFS}"
-			(at 121.7772 58.42 0)
+		(at 125.73 54.61 180)
+		(fields_autoplaced yes)
+		(effects
+			(font
+				(size 1.27 1.27)
+			)
+			(justify right)
+		)
+		(property "Intersheetrefs" "${INTERSHEET_REFS}"
+			(at 119.2372 54.61 0)
 			(effects
 				(font
@@
 	(global_label "VCC"
 		(shape input)
-		(at 142.24 44.45 90)
-		(fields_autoplaced yes)
-		(effects
-			(font
-				(size 1.27 1.27)
-			)
-			(justify left)
-		)
-		(property "Intersheetrefs" "${INTERSHEET_REFS}"
-			(at 142.24 37.8362 90)
+		(at 139.7 40.64 90)
+		(fields_autoplaced yes)
+		(effects
+			(font
+				(size 1.27 1.27)
+			)
+			(justify left)
+		)
+		(property "Intersheetrefs" "${INTERSHEET_REFS}"
+			(at 139.7 34.0262 90)
 			(effects
 				(font
@@
 	(global_label "SDA"
 		(shape input)
-		(at 128.27 54.61 180)
-		(fields_autoplaced yes)
-		(effects
-			(font
-				(size 1.27 1.27)
-			)
-			(justify right)
-		)
-		(property "Intersheetrefs" "${INTERSHEET_REFS}"
-			(at 121.7167 54.61 0)
+		(at 125.73 50.8 180)
+		(fields_autoplaced yes)
+		(effects
+			(font
+				(size 1.27 1.27)
+			)
+			(justify right)
+		)
+		(property "Intersheetrefs" "${INTERSHEET_REFS}"
+			(at 119.1767 50.8 0)
 			(effects
 				(font
@@
 	(global_label "INT to 328p(PD2)"
 		(shape input)
-		(at 151.13 59.69 0)
-		(fields_autoplaced yes)
-		(effects
-			(font
-				(size 1.27 1.27)
-			)
-			(justify left)
-		)
-		(property "Intersheetrefs" "${INTERSHEET_REFS}"
-			(at 171.0484 59.69 0)
+		(at 148.59 55.88 0)
+		(fields_autoplaced yes)
+		(effects
+			(font
+				(size 1.27 1.27)
+			)
+			(justify left)
+		)
+		(property "Intersheetrefs" "${INTERSHEET_REFS}"
+			(at 168.5084 55.88 0)
 			(effects
 				(font
@@
 	(symbol
 		(lib_id "LCustom:Gyro_Absolute_BNO055")
-		(at 139.7 58.42 0)
+		(at 137.16 54.61 0)
 		(unit 1)
 		(exclude_from_sim no)
@@
 		(fields_autoplaced yes)
 		(property "Reference" "U2"
-			(at 141.8433 71.12 0)
+			(at 139.3033 67.31 0)
 			(effects
 				(font
@@
 		)
 		(property "Value" "Gyro_Absolute_BNO055"
-			(at 141.8433 73.66 0)
+			(at 139.3033 69.85 0)
 			(effects
 				(font
@@
 		)
 		(property "Footprint" ""
-			(at 139.7 58.42 0)
+			(at 137.16 54.61 0)
 			(effects
 				(font
@@
 		)
 		(property "Datasheet" ""
-			(at 139.7 58.42 0)
+			(at 137.16 54.61 0)
 			(effects
 				(font
@@
 		)
 		(property "Description" ""
-			(at 139.7 58.42 0)
-			(effects
-				(font
+			(at 137.16 54.61 0)
+			(effects
+				(font
